File: eval-board/pmu.kicad_sch (KiCad schematic)
At the start: 0 parts

Commit message: 5v buck
Parts:
- added C1: 10u, symbol Device:C
- added C2, C3: 100n, symbol Device:C
- added C4, C5: 22u, symbol Device:C
- added C6: 75p, symbol Device:C
- added L1: 10u, symbol Device:L_Iron
- added R1: 511k, symbol Device:R
- added R2: 105k, symbol Device:R
- added R3: 49R9, symbol Device:R
- added R4: 100k, symbol Device:R
- added R5: 13k3, symbol Device:R
- added U1: TPS54302, Package_TO_SOT_SMD:SOT-23-6, symbol Regulator_Switching:TPS54302
Connections:
- new net: C3.2, L1.1, U1.2 (SW)
- new net: R1.2, R2.1, U1.5 (EN)
- new net: C3.1, U1.6 (BOOT)
- new net: C6.1, R3.2, R4.1
- new net: C6.2, R4.2, R5.1, U1.4 (FB)
- new net +5V: C4.1, C5.1, L1.2, R3.1
- new net GND: C1.2, C2.2, C4.2, C5.2, R2.2, R5.2, U1.1 (GND)
- new net VIN: C1.1, C2.1, R1.1, U1.3 (VIN)

Commit message: pmu schematic
Parts:
- added C10, C12: 100n, symbol Device:C
- added C11, C7, C8, C9: 1u, symbol Device:C
- added U2: LP5907MFX-3.3, Package_TO_SOT_SMD:SOT-23-5, symbol Regulator_Linear:LP5907MFX-3.3
- added U3: LD39050PU33R, Package_SON:WSON-6-1EP_3x3mm_P0.95mm, symbol JLCImport:LD39050PU33R
Connections:
- net +5V: now also C10.1, C7.1, C9.1, U2.1 (IN), U2.3 (EN), U3.1 (EN), U3.6 (VIN)
- net GND: now also C10.2, C11.2, C12.2, C7.2, C8.2, C9.2, U2.2 (GND), U3.2 (GND), U3.7 (EXP)
- new net +3V3A: C8.1, U2.5 (OUT)
- new net +3V3D: C11.1, C12.1, U3.4 (VOUT)
- new net +3V3D_PG: U3.3 (PG)

Commit message: imu0 - lsm6dso
Connections:
- no-connect marks 0 -> 1
