File: eval-board/baro.kicad_sch (KiCad schematic)
At the start: 0 parts

Commit message: imu1, baro, mag
Parts:
- added U6: BMP388, JLCImport:BMP388, symbol JLCImport:BMP388
Connections:
- new net +3V3A: U6.10 (VDD)
- new net +3V3D: U6.1 (VDDIO), U6.6 (CSB)
- new net GND: U6.3 (VSS), U6.5 (SDO), U6.8 (VSS), U6.9 (VSS)
- new net INT: U6.7 (INT)
- new net SCL: U6.2 (SCK)
- new net SDA: U6.4 (SDI)
Other:
- note added: "I2C Address: 0x76"
