File: eval-board/imu0.kicad_sch (KiCad schematic)
At the start: 0 parts

Commit message: imu0 - lsm6dso
Parts:
- added C13, C14: 100n, symbol Device:C
- added U4: LSM6DSOTR, Package_LGA:Bosch_LGA-14_3x2.5mm_P0.5mm, symbol JLCImport:LSM6DSOTR
Connections:
- new net +3V3A: C14.1, U4.8 (VDD)
- new net +3V3D: C13.1, U4.5 (VDDIO)
- new net CS: U4.12 (CS)
- new net GND: C13.2, C14.2, U4.2 (SDX), U4.3 (SCX), U4.6 (GND), U4.7 (GND)
- new net INT1: U4.4 (INT1)
- new net INT2: U4.9 (INT2)
- new net SCL: U4.13 (SCL)
- new net SDIO: U4.14 (SDA)
- no-connect marks 0 -> 3

Commit message: imu1, baro, mag
Connections:
- net SCL renamed SCLK
Changed lines of the file:
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@@
 		)
 	)
-	(hierarchical_label "SCL"
+	(hierarchical_label "SCLK"
 		(shape input)
 		(at 166.37 59.69 0)
