File: eval-board/imu1.kicad_sch (KiCad schematic)
At the start: 0 parts

Commit message: imu1, baro, mag
Parts:
- added C15, C16: 100n, symbol Device:C
- added U5: BMI270, Package_LGA:Bosch_LGA-14_3x2.5mm_P0.5mm, symbol JLCImport:BMI270
Connections:
- new net +3V3A: C16.1, U5.8 (VDD)
- new net +3V3D: C15.1, U5.5 (VDDIO)
- new net CS: U5.12 (CSB)
- new net GND: C15.2, C16.2, U5.6 (GNDIO), U5.7 (GND)
- new net INT1: U5.4 (INT1)
- new net INT2: U5.9 (INT2)
- new net SCLK: U5.13 (SCX)
- new net SDIO: U5.14 (SDX)
- no-connect marks 0 -> 5
