File: eval-board/mag.kicad_sch (KiCad schematic)
At the start: 0 parts

Commit message: imu1, baro, mag
Parts:
- added C17: 4u7, symbol Device:C
- added U7: QMC5883P, Package_LGA:LGA-16_3x3mm_P0.5mm, symbol JLCImport:QMC5883P
Connections:
- new net: C17.1, U7.10 (C1)
- new net +3V3D: U7.2 (VDD)
- new net GND: C17.2, U7.11 (GND), U7.9 (GND)
- new net SCL: U7.1 (SCK)
- new net SDA: U7.16 (SDA)
- no-connect marks 0 -> 10
Other:
- note added: "I2C Address: 0x2c"
