File: eval-board/fcu.kicad_sch (KiCad schematic)
At the start: 0 parts

Commit message: fcu serial
Parts:
- added U8: STM32F405RGTx, Package_QFP:LQFP-64_10x10mm_P0.5mm, symbol MCU_ST_STM32F4:STM32F405RGTx
Connections:
- new net: U8.18 (VSS), U8.63 (VSS)
- new net I2C0_SCL: U8.58 (PB6)
- new net I2C0_SDA: U8.59 (PB7)
- new net I2C1_SCL: U8.29 (PB10)
- new net I2C1_SDA: U8.30 (PB11)
- new net PWM0_CH0: U8.37 (PC6)
- new net PWM0_CH1: U8.38 (PC7)
- new net PWM0_CH2: U8.39 (PC8)
- new net PWM0_CH3: U8.40 (PC9)
- new net PWM1_CH0: U8.14 (PA0)
- new net PWM1_CH1: U8.15 (PA1)
- new net SPI0_CS0: U8.24 (PC4)
- new net SPI0_CS1: U8.25 (PC5)
- new net SPI0_MISO: U8.22 (PA6)
- new net SPI0_MOSI: U8.23 (PA7)
- new net SPI0_SCLK: U8.21 (PA5)
- new net SPI1_CS0: U8.33 (PB12)
- new net SPI1_MISO: U8.35 (PB14)
- new net SPI1_MOSI: U8.36 (PB15)
- new net SPI1_SCLK: U8.34 (PB13)
- new net SPI2_CS0: U8.50 (PA15)
- new net SPI2_MISO: U8.52 (PC11)
- new net SPI2_MOSI: U8.53 (PC12)
- new net SPI2_SCLK: U8.51 (PC10)
- new net UART0_RX: U8.43 (PA10)
- new net UART0_TX: U8.42 (PA9)
- new net UART1_RX: U8.17 (PA3)
- new net UART1_TX: U8.16 (PA2)
Other:
- note added: "I2C1"
- note added: "I2C2"
- note added: "SPI1"
- note added: "SPI2"
- note added: "SPI3"
- note added: "TIM2 CH1 CH2"
- note added: "TIM3 CH1-4"
- note added: "USART1"
- note added: "USART2"
